Commit message: added "sea floor plane and correct orientation with lidar"

File: src/vrx/vrx_urdf/wamv_gazebo/urdf/components/wamv_3d_lidar.xacro (robot description, xacro)
@@ -120,5 +120,5 @@
     <xacro:property name="post_to_lidar_x" value="${post_to_post_arm_x+post_arm_to_lidar_x}"/>
     <joint name="${namespace}/base_to_${name}_post_joint" type="fixed">
-      <origin xyz="${x-(post_to_lidar_x)*cos(post_Y)} ${y-(post_to_lidar_x)*sin(post_Y)} ${post_z}" rpy="0 0 ${post_Y}" />
+      <origin xyz="${x-(post_to_lidar_x)*cos(post_Y)} ${y-(post_to_lidar_x)*sin(post_Y)} ${0.79}" rpy="0 0 ${post_Y}" />
       <parent link="${namespace}/base_link" />
       <child link="${namespace}/${name}_post_link" />
@@ -126,5 +126,5 @@
     <!-- Sensor post to sensor post arm joint -->
     <joint name="${namespace}/${name}_post_to_${name}_post_arm_joint" type="fixed">
-      <origin xyz="${post_to_post_arm_x} 0 ${z-post_z-post_arm_to_lidar_z}" rpy="0 0 0" />
+      <origin xyz="${post_to_post_arm_x} 0 ${-0.7}" rpy="0 0 0" />
       <parent link="${namespace}/${name}_post_link" />
       <child link="${namespace}/${name}_post_arm_link" />
@@ -132,5 +132,5 @@
     <!-- Sensor post arm to lidar joint -->
     <joint name="${namespace}/${name}_post_arm_to_${name}_joint" type="fixed">
-      <origin xyz="${post_arm_to_lidar_x} 0 ${post_arm_to_lidar_z}" rpy="${R} ${P} ${Y-post_Y}" />
+      <origin xyz="${post_arm_to_lidar_x} 0 ${-post_arm_to_lidar_z}" rpy="${R + 1.57} ${P + 1.57} ${Y-post_Y}" />
       <parent link="${namespace}/${name}_post_arm_link" />
       <child link="${namespace}/${name}_link" />
