Commit message: correct lidar, Map topic fulling

File: src/vrx/vrx_urdf/wamv_description/urdf/wamv_base.urdf.xacro (robot description, xacro)
@@ -165,6 +165,6 @@
   <parent link="${namespace}/base_link"/>
   <child link="laser_down_link"/>
-  <!-- Adjust the xyz position to your desired sensor placement -->
-  <origin xyz="0 0 -0.1" rpy="0 0 0"/>
+  <!-- Rotated 90 degrees about X to point scan directly down -->
+  <origin xyz="0 0 -0.1" rpy="1.5708 0 0"/>
 </joint>
 <!-- Gazebo sensor definition -->
@@ -176,12 +176,12 @@
       <scan>
         <horizontal>
-          <samples>1</samples>
-          <min_angle>0</min_angle>
-          <max_angle>0</max_angle>
+          <samples>360</samples>
+          <min_angle>-3.14159</min_angle>
+          <max_angle>3.14159</max_angle>
         </horizontal>
       </scan>
       <range>
         <min>0.1</min>
-        <max>5.0</max>
+        <max>20.0</max>
       </range>
     </ray>
@@ -191,8 +191,36 @@
         <remapping>~/out:=laser_down/scan</remapping>
       </ros>
-      <frame_name>laser_down_link</frame_name>
+      <frame_name>wamv/wamv/base_link</frame_name>
       <output_type>sensor_msgs/LaserScan</output_type>
     </plugin>
   </sensor>
 </gazebo>
+<!-- Seafloor (visible box) -->
+<gazebo reference="world">
+  <model name="seafloor_box">
+    <static>true</static>
+    <pose>0 0 0 0 0 0</pose>
+    <link name="link">
+      <collision name="collision">
+        <geometry>
+          <box>
+            <size>5000 5000 1</size>
+          </box>
+        </geometry>
+      </collision>
+      <visual name="visual">
+        <geometry>
+          <box>
+            <size>5000 5000 1</size>
+          </box>
+        </geometry>
+        <material>
+          <ambient>0.2 0.4 0.2 1</ambient>
+          <diffuse>0.2 0.4 0.2 1</diffuse>
+          <specular>0.1 0.1 0.1 1</specular>
+        </material>
+      </visual>
+    </link>
+  </model>
+</gazebo>
 </robot>

Commit message: fixed imu base link transform. added imu covarience for EKF, switched format of EKF pipelin

File: src/vrx/vrx_urdf/wamv_description/urdf/wamv_base.urdf.xacro (robot description, xacro)
@@ -107,4 +107,18 @@
       <inertia ixx="120.0" ixy="0.0" ixz="0.0" iyy="393" iyz="0.0" izz="446.0"/>
     </inertial>
+    <!-- IMU mount link -->
+    <link name="${namespace}/imu_wamv_link"/>
+    <joint name="imu_mount_joint" type="fixed">
+      <parent link="${namespace}/base_link"/>
+      <child link="${namespace}/imu_wamv_link"/>
+      <origin xyz="0 0 0" rpy="0 0 0"/>
+    </joint>
+    <!-- IMU sensor link -->
+    <link name="${namespace}/imu_wamv_link/imu_wamv_sensor"/>
+    <joint name="imu_sensor_joint" type="fixed">
+      <parent link="${namespace}/imu_wamv_link"/>
+      <child link="${namespace}/imu_wamv_link/imu_wamv_sensor"/>
+      <origin xyz="0 0 0" rpy="0 0 0"/>
+    </joint>
   </link>
   <gazebo>
